File: HOT_AIRGUN_EXTRADOPE.kicad_sch (KiCad schematic)
At the start: 45 parts, among them J5 Conn_01x04_Socket, J6 Conn_01x05_Pin, J7 Conn_01x02_Socket, J8 Conn_02x05_Counter_Clockwise, J9 Conn_02x03_Counter_Clockwise, SW1 TSB008A2526A, SW2 TSB008A2526A, U10 DB301V-3.5-2P-GN, U11 DB301V-3.5-2P-GN, U12 DB301V-3.5-2P-GN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

Commit message: Finished Routing, Finished Schematic
Yet to add , solderMask
Parts:
- removed TP2: Vref_TPgnd, TestPoint:TestPoint_THTPad_2.0x2.0mm_Drill1.0mm, symbol Connector:TestPoint
- added H1, H2, H3: MountingHole, MountingHole:MountingHole_3.2mm_M3_Pad_Via, symbol Mechanical:MountingHole
- added TP10: GND_TP, TestPoint:TestPoint_THTPad_2.0x2.0mm_Drill1.0mm, symbol Connector:TestPoint
- C11, C12, C13, C14, C15: value 1u -> 100n
- J5: footprint Connector_Wire:SolderWire-0.5sqmm_1x04_P4.6mm_D0.9mm_OD2.1mm_Relief -> Connector_Wire:SolderWire-0.5sqmm_1x04_P4.6mm_D0.9mm_OD2.1mm
- J7: footprint Connector_Wire:SolderWire-0.5sqmm_1x02_P4.6mm_D0.9mm_OD2.1mm_Relief -> Connector_Wire:SolderWire-0.5sqmm_1x02_P4.6mm_D0.9mm_OD2.1mm
Connections:
- net AcLoad1- is gone; now on net NEUT: U12.2
- net AcLoad2- is gone; now on net NEUT: U13.2
- net DC_Load1+ is gone; now on net +24V: U11.1
- net DC_Load2+ is gone; now on net +24V: U10.1
- net DC_Load3+ is gone; now on net +24V: U9.1
- net VREF_2p5 is gone; now on net VREF2p5: R32.1, R33.1, U4.8 (Ref)
- net GND: now also TP10.1
- net ThermocoupleSig1: now also U2.5 (SENSOR_VN); no longer U2.7 (IO35)
- net ThermocoupleSig2: now also U2.4 (SENSOR_VP); no longer U2.8 (IO32)
- net VREFAtt1: now also U2.8 (IO32); no longer U2.4 (SENSOR_VP)
- net VREFAtt2: now also U2.7 (IO35); no longer U2.5 (SENSOR_VN)
