File: PowerControl.kicad_sch (KiCad schematic)
At the start: 21 parts, among them Q3 BT136-500, Q4 BT136-500, Q5 S9013_C402281, Q6 S9013_C402281, Q7 AO3400_C2938367, Q8 AO3400_C2938367, Q9 AO3400_C2938367, T1 MOC3020M, T2 MOC3020M

Commit message: Finished Routing, Finished Schematic
Yet to add , solderMask
Parts:
- added D2, D4, D5: SD103AW_C181204, EasyEDA:SOD-123_L2.8-W1.8-LS3.7-RD, symbol EasyEDA:SD103AW_C181204
- added D6, D8, D9: LED, LED_SMD:LED_1206_3216Metric_Pad1.42x1.75mm_HandSolder, symbol Device:LED
- added R38, R40, R41: 10k, Resistor_SMD:R_1206_3216Metric_Pad1.30x1.75mm_HandSolder, symbol Device:R
Connections:
- net +24V: now also D2.1 (K), D4.1 (K), D5.1 (K), R38.1, R40.1, R41.1
- net DC_Load1-: now also D2.2 (A), D6.1 (K)
- net DC_Load2-: now also D4.2 (A), D8.1 (K)
- net DC_Load3-: now also D5.2 (A), D9.1 (K)
- new net: D8.2 (A), R40.2
- new net: D9.2 (A), R41.2
- new net: D6.2 (A), R38.2
Other:
- note added: "DC Control"
- note removed: "Blower Control"
- moved on the sheet: Q9, R22, R23, R27, R28, R7, R8

Commit message: Fixed Silkscreen, Added production files
Parts:
- renumbered D6 to D3, D5 to D4, D9 to D5, D4 to D6, D8 to D7, Q6 to Q1, Q5 to Q2, Q4 to Q3, Q3 to Q4, Q8 to Q5, Q9 to Q6, R4 to R10, R3 to R11, R6 to R12, R5 to R13, R7 to R14, R8 to R15, R27 to R16, R38 to R17, R28 to R18, R41 to R19, R22 to R20, R23 to R21, R40 to R22, R1 to R8, R2 to R9, T2 to T1, T1 to T2

Commit message: Key Fixes and upgrade to V0.1
Design reliance on dedicated thermocouple interface chip instead of calibrating adc and differential amplifier ; Neater routing ; Logos ; High voltage spacing for AC part
Parts:
- added HS1, HS2: Heatsink_Pad, LibMain:TO-220 HeatPad, symbol Mechanical:Heatsink_Pad
- D5: renamed from D3; LCSC Part (none) -> C965822
- D7: renamed from D5; LCSC Part (none) -> C965822
- D9: renamed from D7; LCSC Part (none) -> C965822
- Q3, Q4: LCSC Part (none) -> C916781
- R10: renamed from R11; value 1K -> 1k; LCSC Part (none) -> C2907440
- R11: renamed from R12; LCSC Part (none) -> C2907486
- R12: renamed from R13; LCSC Part (none) -> C2907486
- R13: renamed from R14; LCSC Part (none) -> C2907528
- R14: renamed from R15; LCSC Part (none) -> C17902
- R15: renamed from R16; LCSC Part (none) -> C2907528
- R16: renamed from R17; LCSC Part (none) -> C17902
- R17: renamed from R18; LCSC Part (none) -> C17902
- R18: renamed from R19; LCSC Part (none) -> C17902
- R19: renamed from R20; LCSC Part (none) -> C2907528
- R20: renamed from R21; LCSC Part (none) -> C17902
- R21: renamed from R22; LCSC Part (none) -> C17902
- R7: renamed from R8; LCSC Part (none) -> C17902
- R8: renamed from R9; LCSC Part (none) -> C17902
- R9: renamed from R10; value 1K -> 1k; LCSC Part (none) -> C2907440
- renumbered D2 to D4, D4 to D6, D6 to D8
Connections:
- no-connect marks 4 -> 6
Other:
- moved on the sheet: D6, D7, Q6, R15, R17, R18
